File: UA18_Datalogger/UA18_shield.brd (EAGLE design)
At the start: 87.6 x 74.9 mm, 5 parts, among them IC1 4067D, IC2 4067D, U2 ARDUINOR3-DIMENSION

Commit message: finished datalogger
Connections:
- removed net D2: U$1.3,2A
- removed net D3: U$1.3,3A
- removed net D4: U$1.3,4A
- removed net D5: U$1.3,5A
- removed net P1: U$1.2,4A
- removed net P2: U$1.2,5A
- net 5V: now also U$1.3,2A, U$1.3,3A, U$1.3,4A, U$1.3,5A; no longer U$1.2,3A
- net GND: now also U$1.2,3A, U$1.2,4A, U$1.2,5A
Routing:
- net GND: track 83.9 -> 117.2 mm
- net 5V: track 107.8 -> 123.6 mm
Other:
- outline, holes or cut-outs redrawn
